File: Node/node.brd (EAGLE design)
At the start: 76.2 x 33.9 mm, 126 parts, among them J1 U.FL, J2 USBSMD, J3 CORTEX_DEBUGPTH, U1 MCP73871, U2 DW1000-I, U3 TPS61090RSAR, U4 ATMEGA328, U5 LSM303C, U6 LM3880, X2 332-02, Y2 8MHZ

Commit message: Initial commit with new schematic and general board layout.
Parts:
- removed 3, CPRST, G, I, O, R, S: TPSQTP08R, testpad:TP08R
- removed C36: 4.7uF, SparkFun-Capacitors:0805-CAP
- removed C37: 2uF, SparkFun-Capacitors:0805-CAP
- removed C38: 1uF, SparkFun-Capacitors:0805-CAP
- removed FTDI: (no value), adafruit:1X06-BIGLOCK
- removed J3: CORTEX_DEBUGPTH, SparkFun-Connectors:2X5-PTH-1.27MM
- removed JP1: (no value), SparkFun-Connectors:1X04
- removed RST: 10k, resistor:R0805
- removed RST1: 4.7K, resistor:R0805
- removed RXOK1, SFD1: (no value), SparkFun-LED:LED-0603
- removed U$12: 23A640, MainLib:SOIC-8
- removed U$8: CP2105, MainLib:QFN50P400X400X80-25N
- removed Y2: 8MHZ, SparkFun-FreqCtrl:RESONATOR-SMD
- added C43: 10uF, microbuilder:0805-NO
- added C44: 22pF, microbuilder:0603-NO
- added I2C, UART: (no value), SparkFun-Connectors:1X04
- added J5: CORTEX_DEBUGPTH, SparkFun-Connectors:2X5-PTH-1.27MM
- added L4, L5: RED, microbuilder:CHIPLED_0805_NOOUTLINE
- added L6: GREEN, microbuilder:CHIPLED_0805_NOOUTLINE
- added R31: 470, SparkFun-Resistors:0603-RES
- added R32, R34: 47K, SparkFun-Resistors:0603-RES
- added R33: 10K, SparkFun-Resistors:0603-RES
- added SJ3: (no value), jumper:SJ
- added SW2: SPST_TACT-KMR2, adafruit:KMR2
- added X3: 32.768, adafruit2:XTAL3215
- C1: value 0.1uF -> 1uF; device SparkFun-Capacitors:0805-CAP -> microbuilder:0603-NO
- C2: value 0.1uF -> 22pF; device SparkFun-Capacitors:0805-CAP -> microbuilder:0603-NO
- R1, R2, R3: device resistor:R0805 -> SparkFun-Resistors:0603-RES
- R13, R14, R15, R16, R17, R20, R22, R24, R25, THERM: device SparkFun-Passives:0805 -> SparkFun-Resistors:0603-RES
- R21, R23: device SparkFun-Passives:0402-RES -> SparkFun-Resistors:0603-RES
- U4: value ATMEGA328 -> ATSAMD21G-A; device SparkFun:TQFP32-08 -> samd21:TQFP-48
- moved C2 14.3 mm to (47.7, 19.2), turned to 270 degrees
- moved R27 12.1 mm to (57.0, 10.9), turned to 90 degrees
- moved R26 11.4 mm to (55.2, 10.9), turned to 90 degrees
- moved X2 10.7 mm to (40.9, 31.2), turned to 90 degrees
- moved R21 8.44 mm to (7.59, 28.9)
- moved SJ1 7.58 mm to (26.4, 11.2), turned to 270 degrees
- moved C1 7.40 mm to (43.8, 13.5), turned to 315 degrees
- moved U4 6.23 mm to (38.6, 18.3), turned to 225 degrees
- moved R23 4.13 mm to (23.4, 29.0)
- moved TP2 3.31 mm to (28.4, 13.2)
- moved TP1 3.06 mm to (28.4, 14.5)
- moved TP3-OTP 2.65 mm to (28.4, 15.7)
- moved THERM 1.12 mm to (43.8, 22.7), turned to 315 degrees
- moved R15 1.02 mm to (72.1, 15.0)
- moved R24 0.76 mm to (53.5, 13.8)
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- renumbered JP2 to SPI
Connections:
- removed net !SRAMCS: U$12.1, U4.12
- removed net !SRAMHOLD: U$12.7, U4.24
- removed net A3: U4.26
- removed net A6: U4.19
- removed net A7: U4.22
- removed net CPVIO: C37.2, R21.2, R23.2, RST1.2, U$8.5, U$8.6
- removed net D4: U4.2
- removed net DTR: C1.1, FTDI.6, U$8.23
- removed net N$19: CPRST.TP, RST1.1, U$8.9
- removed net N$29: C36.1, U$8.16
- removed net RESET: C1.2, R.TP, RST.1, U4.29, X2.2
- removed net RX_LED: SFD1.C, U$8.14
- removed net TX_LED: RXOK1.C, U$8.15
- new net !RESET: R33.2, SJ3.2, SW2.1, SW2.3, U4.40, X2.2
- new net A0: U4.3
- new net A1: U4.7
- new net A2: U4.8
- new net A4: U4.10
- new net A5: U4.47
- new net D0: U4.16
- new net D1: U4.15
- new net D11: U4.25
- new net D12: U4.28
- new net D13LED: R21.1, U4.26
- new net LIPOADC: R32.1, R34.2, U4.9
- new net N$33: C1.1, U4.43
- new net N$35: C2.1, U4.2, X3.P$1
- new net N$36: C44.1, U4.1, X3.P$2
- new net RXLED: R23.1, U4.48
- new net SWCLK: J5.4, U4.45
- new net SWDIO: J5.2, U4.46
- new net TXLED: R31.1, U4.39
- net !EXTCS: now also U4.12; no longer U4.25
- net !SPICS: now also U4.27; no longer U4.14
- net 3.3V: now also C43.1, I2C.2, J5.1, L5.A, L6.A, R33.1, SPI.2, U4.17, U4.36, U4.44, UART.2; no longer 3.TP, C38.1, FTDI.3, JP1.2, RST.2, SPI.1, U$12.8, U4.18, U4.4
- net AREF: now also U4.4; no longer C2.1, U4.20
- net BLU: now also U4.30; no longer U4.1
- net D+: now also U4.34; no longer U$8.3
- net D-: now also U4.33; no longer U$8.4
- net DWRST: now also U4.11; no longer U4.13
- net EXTON: now also U4.13; no longer U4.23
- net GND: now also C1.2, C43.2, C44.2, I2C.1, J5.3, J5.5, J5.9, L4.C, R34.1, SPI.1, SW2.2, SW2.4, U4.18, U4.35, U4.42, UART.1; no longer C36.2, C37.1, C38.2, FTDI.1, FTDI.2, G.TP, JP1.1, SPI.2, U$12.4, U$8.2, U$8.25, U4.21, U4.3, Y2.2
- net GRN: now also U4.24; no longer U4.9
- net IQR: now also U4.23; no longer U4.32
- net MISO: now also U4.21; no longer I.TP, U$12.2, U4.16
- net MOSI: now also U4.19; no longer O.TP, U$12.5, U4.15
- net N$1: now also J5.10, SJ3.1; no longer U4.8, Y2.3
- net N$31: now also L4.A, R21.2; no longer R21.1, RXOK1.A
- net N$32: now also L6.C, R31.2; no longer R23.1, SFD1.A
- net N$9: now also L5.C, R23.2; no longer U4.7, Y2.1
- net RED: now also U4.14; no longer U4.10
- net RXD: now also U4.38, UART.4; no longer FTDI.4, U$8.21, U4.30
- net SCK: now also U4.20; no longer S.TP, U$12.6, U4.17
- net SCL: now also I2C.4, U4.32; no longer JP1.4, U4.28
- net SDA: now also I2C.3, U4.31; no longer JP1.3, U4.27
- net TXD: now also U4.37, UART.3; no longer FTDI.5, U$8.20, U4.31
- net VBUS: no longer U$8.7, U$8.8
- net VLIPO: now also R32.2
- net WAKEUP: now also U4.29; no longer U4.11
Routing:
- net !RESET: track 0.00 -> 76.7 mm, vias 0 -> 3
- net DTR: track 36.2 -> 0.00 mm, vias 2 -> 0
- net D13LED: track 0.00 -> 35.0 mm
- net RESET: track 33.8 -> 0.00 mm, vias 3 -> 0
- net RXLED: track 0.00 -> 31.6 mm, vias 0 -> 2
- net TXLED: track 0.00 -> 30.6 mm, vias 0 -> 2
- net CPVIO: track 29.1 -> 0.00 mm, vias 2 -> 0
- net !SRAMCS: track 27.4 -> 0.00 mm, vias 2 -> 0
- net TXD: track 34.3 -> 10.2 mm
- net TX_LED: track 24.0 -> 0.00 mm, vias 2 -> 0
- net RX_LED: track 23.3 -> 0.00 mm, vias 2 -> 0
- net SWCLK: track 0.00 -> 22.8 mm
- net D+: track 23.5 -> 45.8 mm, vias 1 -> 2
- net D-: track 23.7 -> 44.1 mm, vias 1 -> 2
- net SWDIO: track 0.00 -> 20.3 mm
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Other:
- board text added: "3.3V"
- board text added: "GND"
- board text added: "SPI"
- board text added: "UART"
